Commit message: Adding option to scale the added-mass, linear damping and quadratic damping matrices. Adding ROS service to return all hydrodynamic model parameters for a link.
Signed-off-by: Musa Morena Marcusso Manhães <Musa.Marcusso@de.bosch.com>

File: uuv_descriptions/models/rexrov/robots/rexrov_default.xacro (robot description, xacro)
@@ -15,8 +15,16 @@
   <xacro:arg name="debug" default="0"/>
   <xacro:arg name="namespace" default="rexrov"/>
+  <xacro:arg name="scaling_added_mass" default="1"/>
+  <xacro:arg name="scaling_linear_damp" default="1"/>
+  <xacro:arg name="scaling_quad_damping" default="1"/>
   <!-- Include the ROV macro file -->
   <xacro:include filename="$(find uuv_descriptions)/models/rexrov/urdf/rexrov_base.xacro"/>
   <!-- Create the rexrov -->
-  <xacro:rexrov_base namespace="$(arg namespace)" debug="$(arg debug)"/>
+  <xacro:rexrov_base
+    namespace="$(arg namespace)"
+    debug="$(arg debug)"
+    scaling_added_mass="$(arg scaling_added_mass)"
+    scaling_linear_damp="$(arg scaling_linear_damp)"
+    scaling_quad_damping="$(arg scaling_quad_damping)"/>
   <!-- Joint state publisher plugin -->
   <xacro:default_joint_state_publisher namespace="$(arg namespace)" update_rate="500"/>

File: uuv_descriptions/models/rexrov/robots/rexrov_oberon4.xacro (robot description, xacro)
@@ -15,9 +15,17 @@
   <xacro:arg name="debug" default="0"/>
   <xacro:arg name="namespace" default="rexrov"/>
+  <xacro:arg name="scaling_added_mass" default="1"/>
+  <xacro:arg name="scaling_linear_damp" default="1"/>
+  <xacro:arg name="scaling_quad_damping" default="1"/>
   <!-- Include the ROV macro file -->
   <xacro:include filename="$(find uuv_descriptions)/models/rexrov/urdf/rexrov_base.xacro"/>
   <xacro:include filename="$(find oberon4_description)/robots/oberon4_default.xacro" />
   <!-- Create the ROV -->
-  <xacro:rexrov_base namespace="$(arg namespace)" debug="$(arg debug)"/>
+  <xacro:rexrov_base
+    namespace="$(arg namespace)"
+    debug="$(arg debug)"
+    scaling_added_mass="$(arg scaling_added_mass)"
+    scaling_linear_damp="$(arg scaling_linear_damp)"
+    scaling_quad_damping="$(arg scaling_quad_damping)"/>
   <xacro:oberon4 namespace="oberon4" parent="$(arg namespace)/base_link">
     <origin xyz="1.3 0.5 -0.615" rpy="0 0 0"/>

File: uuv_descriptions/models/rexrov/robots/rexrov_oberon_arms.xacro (robot description, xacro)
@@ -15,4 +15,7 @@
   <xacro:arg name="debug" default="0"/>
   <xacro:arg name="namespace" default="rexrov"/>
+  <xacro:arg name="scaling_added_mass" default="1"/>
+  <xacro:arg name="scaling_linear_damp" default="1"/>
+  <xacro:arg name="scaling_quad_damping" default="1"/>
   <!-- Include the ROV macro file -->
   <xacro:include filename="$(find uuv_descriptions)/models/rexrov/urdf/rexrov_base.xacro"/>
@@ -20,5 +23,10 @@
   <xacro:include filename="$(find oberon_description)/robots/oberon_parallel.xacro" />
   <!-- Create the ROV -->
-  <xacro:rexrov_base namespace="$(arg namespace)" debug="$(arg debug)"/>
+  <xacro:rexrov_base
+    namespace="$(arg namespace)"
+    debug="$(arg debug)"
+    scaling_added_mass="$(arg scaling_added_mass)"
+    scaling_linear_damp="$(arg scaling_linear_damp)"
+    scaling_quad_damping="$(arg scaling_quad_damping)"/>
   <xacro:oberon namespace="oberon" parent="$(arg namespace)/base_link">
     <origin xyz="1.3 -0.5 -0.615" rpy="0 0 0"/>

File: uuv_descriptions/models/rexrov/robots/rexrov_oberon_dummy.xacro (robot description, xacro)
@@ -15,4 +15,7 @@
   <xacro:arg name="debug" default="0"/>
   <xacro:arg name="namespace" default="rexrov"/>
+  <xacro:arg name="scaling_added_mass" default="1"/>
+  <xacro:arg name="scaling_linear_damp" default="1"/>
+  <xacro:arg name="scaling_quad_damping" default="1"/>
   <!-- Include the ROV macro file -->
   <xacro:include filename="$(find uuv_descriptions)/models/rexrov/urdf/rexrov_base.xacro"/>
@@ -20,4 +23,10 @@
   <!-- Create the ROV -->
   <xacro:rexrov_base namespace="$(arg namespace)" debug="$(arg debug)"/>
+  <xacro:rexrov_base
+    namespace="$(arg namespace)"
+    debug="$(arg debug)"
+    scaling_added_mass="$(arg scaling_added_mass)"
+    scaling_linear_damp="$(arg scaling_linear_damp)"
+    scaling_quad_damping="$(arg scaling_quad_damping)"/>
   <xacro:oberon namespace="oberon" parent="$(arg namespace)/base_link">
     <origin xyz="1.3 -0.5 -0.615" rpy="0 0 0"/>

File: uuv_descriptions/models/rexrov/robots/rexrov_oberon_parallel.xacro (robot description, xacro)
@@ -15,9 +15,17 @@
   <xacro:arg name="debug" default="0"/>
   <xacro:arg name="namespace" default="rexrov"/>
+  <xacro:arg name="scaling_added_mass" default="1"/>
+  <xacro:arg name="scaling_linear_damp" default="1"/>
+  <xacro:arg name="scaling_quad_damping" default="1"/>
   <!-- Include the ROV macro file -->
   <xacro:include filename="$(find uuv_descriptions)/models/rexrov/urdf/rexrov_base.xacro"/>
   <xacro:include filename="$(find oberon_description)/robots/oberon_parallel.xacro" />
   <!-- Create the ROV -->
-  <xacro:rexrov_base namespace="$(arg namespace)" debug="$(arg debug)"/>
+  <xacro:rexrov_base
+    namespace="$(arg namespace)"
+    debug="$(arg debug)"
+    scaling_added_mass="$(arg scaling_added_mass)"
+    scaling_linear_damp="$(arg scaling_linear_damp)"
+    scaling_quad_damping="$(arg scaling_quad_damping)"/>
   <xacro:oberon namespace="oberon" parent="$(arg namespace)/base_link">
     <origin xyz="1.3 -0.5 -0.615" rpy="0 0 0"/>

File: uuv_descriptions/models/rexrov/robots/rexrov_sonar.xacro (robot description, xacro)
@@ -15,8 +15,16 @@
   <xacro:arg name="debug" default="0"/>
   <xacro:arg name="namespace" default="rexrov"/>
+  <xacro:arg name="scaling_added_mass" default="1"/>
+  <xacro:arg name="scaling_linear_damp" default="1"/>
+  <xacro:arg name="scaling_quad_damping" default="1"/>
   <!-- Include the ROV macro file -->
   <xacro:include filename="$(find uuv_descriptions)/models/rexrov/urdf/rexrov_base.xacro"/>
   <!-- Create the rexrov -->
-  <xacro:rexrov_base namespace="$(arg namespace)" debug="$(arg debug)"/>
+  <xacro:rexrov_base
+    namespace="$(arg namespace)"
+    debug="$(arg debug)"
+    scaling_added_mass="$(arg scaling_added_mass)"
+    scaling_linear_damp="$(arg scaling_linear_damp)"
+    scaling_quad_damping="$(arg scaling_quad_damping)"/>
   <xacro:forward_multibeam_sonar_m450_130 namespace="$(arg namespace)" parent_link="$(arg namespace)/base_link">
     <origin xyz="1.4 0 0.65" rpy="0 0 0"/>

File: uuv_descriptions/models/rexrov/urdf/rexrov_base.xacro (robot description, xacro)
@@ -79,5 +79,6 @@
     </gazebo>
   </xacro:macro>
-  <xacro:macro name="rexrov_base" params="namespace debug">
+  <xacro:macro name="rexrov_base" params="namespace debug scaling_added_mass
+    scaling_linear_damp scaling_quad_damping">
     <!-- base_link according to ROS conventions: x forward, z up -->
     <link name="${namespace}/base_link">
@@ -149,8 +150,11 @@
                 -7.8033 62.726 10.775 21.019 -1.1162 224.32
             </added_mass>
+            <added_mass_scaling>${scaling_added_mass}</added_mass_scaling>
             <!-- Linear damping: see p.31 in Berg2012 -->
             <linear_damping>-74.82 -69.48 -728.4 -268.8 -309.77 -105</linear_damping>
+            <linear_damping_scaling>${scaling_linear_damp}</linear_damping_scaling>
             <!-- Non-linear damping: see p.30 in Berg2012 -->
             <quadratic_damping>-748.22 -992.53 -1821.01 -672 -774.44 -523.27</quadratic_damping>
+            <quad_damping_scaling>${scaling_quad_damping}</quad_damping_scaling>
           </hydrodynamic_model>
         </link>
